File: hardware/KiCad/Carte_Volant_v21.sch (KiCad schematic (older format))
At the start: 51 parts, among them J1 RJ45_CANBUS_copy, J2 Conn_01x03, J3 Conn_01x40, J7 Conn_01x03, Q2 FDN337N, U1 TSR_1-2450, U2 STM32H103-OlimexBoard, U3 MCP2561-E-SN

Commit message: errata correction : RJ45 connector + common volatge source + added 3d models + logo + ...
Parts:
- C2: value C -> 105
- J1: value RJ45_CANBUS_copy -> RJ45_CANBUS
- U2: symbol TIM_Microcontrollers_V5:STM32H103-OlimexBoard -> Carte_Volant_v21-rescue:STM32H103-OlimexBoard-TIM_Microcontrollers_V5
- renumbered Alim_12v2 to Alim_12V1, Alim_12v1 to Alim_5V1
Connections:
- net +12V: now also Alim_12V1.1, J1.8 (+12V); no longer Alim_12V1.2, U1.1 (Vin)
- net +3V3: now also C4.2; no longer C4.1
- net GND: now also C4.1, JP_BS1.3 (B); no longer C4.2
- removed net -POWER_ON-OFF: Alim_12V1.1, J1.8 (+12V), J3.2 (Pin_2)
- new net POWER_SWITCH: Alim_12V1.2, J3.2 (Pin_2), U1.1 (Vin)
- no-connect marks 6 -> 3
Other:
- note added: "CAN Transceiver"
- note added: "COMMON VOLTAGE SOURCE \n"
- note added: "HAT SCREEN CONNECTOR\n"
- note added: "MCU"
- note added: "POWER"
- note added: "RAW SCREEN CIRCUITRY\n"
- note added: "WIPER\n"
- note removed: "ALIMENTATION\n"
- note removed: "Transceiver CAN"
- note removed: "wiper\n"
- moved on the sheet: +3, -1, Alim_12V1, Alim_5V1, BUSY1, C10, C11, C12, C13, C14, C2, C3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
